Commit message: Add laser scan and hover on obstacle detection

File: simple_drone_description/urdf/simple_drone.urdf (robot description, URDF)
Before this commit: robot simple_drone, 5 links, 4 joints
Links:
- link base_link: geometry collision mesh filename=file:///home/illia/ros2_ws/install/simple_drone_description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; visual mesh filename=file:///home/illia/ros2_ws/install/simple_drone_description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

File: simple_drone_description/urdf/simple_drone.urdf.xacro (robot description, xacro)
@@ -97,4 +97,35 @@
   </gazebo>
   <!-- Sensors -->
+  <!-- Laser sensor in 100fps -->
+  <gazebo reference="base_link">
+    <sensor name='sensor_ray' type='ray'>
+      <always_on>1</always_on>
+      <visualize>1</visualize>
+      <update_rate>100</update_rate>
+      <pose> 0 0 0 0 0 0 </pose>
+      <ray>
+        <scan>
+          <horizontal>
+            <samples>200</samples>
+            <resolution>1.0</resolution>
+            <min_angle>-0.1</min_angle>
+            <max_angle>0.1</max_angle>
+          </horizontal>
+        </scan>
+        <range>
+          <min>0.10</min>
+          <max>5.0</max>
+        </range>
+      </ray>
+      <plugin name="laser_scan" filename="libgazebo_ros_ray_sensor.so">
+        <ros>
+          <namespace>${mp['namespace']}</namespace>
+        </ros>
+        <output_type>sensor_msgs/LaserScan</output_type>
+        <initial_orientation_as_reference>false</initial_orientation_as_reference>
+        <frame_name>simple_drone/base_link</frame_name>
+      </plugin>
+    </sensor>
+  </gazebo>
   <!-- IMU sensor in 100fps -->
   <gazebo reference="base_link">
@@ -162,5 +193,4 @@
         <ros>
           <namespace>${mp['namespace']}</namespace>
-          <!-- <remapping>~/out:=sonar</remapping> -->
         </ros>
         <frame_name>${mp['namespace']}/sonar_link</frame_name>
